Commit message: first

File: turtlebot3_manipulation_description/ros2_control/turtlebot3_manipulation_system.ros2_control.xacro (robot description, xacro)
@@ -107,6 +107,11 @@
           <param name="max">${pi*0.9}</param>
         </command_interface>
-        <state_interface name="position">
-          <param name="initial_value">0.0</param>
+        <!-- Velocity control -->
+        <command_interface name="velocity">
+          <param name="min">${-pi*1.0}</param>  <!-- Adjust min and max velocity as needed -->
+          <param name="max">${pi*1.0}</param>
+        </command_interface>
+        <state_interface name="position">
+          <param name="initial_value">1.0</param>
         </state_interface>
         <state_interface name="velocity">
@@ -119,4 +124,9 @@
           <param name="max">${pi*0.5}</param>
         </command_interface>
+        <!-- Velocity control -->
+        <command_interface name="velocity">
+          <param name="min">${-pi*1.0}</param>  <!-- Adjust min and max velocity as needed -->
+          <param name="max">${pi*1.0}</param>
+        </command_interface>
         <state_interface name="position">
           <param name="initial_value">0.0</param>
@@ -131,4 +141,9 @@
           <param name="max">${pi*0.44}</param>
         </command_interface>
+        <!-- Velocity control -->
+        <command_interface name="velocity">
+          <param name="min">${-pi*1.0}</param>  <!-- Adjust min and max velocity as needed -->
+          <param name="max">${pi*1.0}</param>
+        </command_interface>
         <state_interface name="position">
           <param name="initial_value">0.0</param>
@@ -142,4 +157,9 @@
           <param name="min">${-pi*0.57}</param>
           <param name="max">${pi*0.65}</param>
+        </command_interface>
+        <!-- Velocity control -->
+        <command_interface name="velocity">
+          <param name="min">${-pi*1.0}</param>  <!-- Adjust min and max velocity as needed -->
+          <param name="max">${pi*1.0}</param>
         </command_interface>
         <state_interface name="position">

File: turtlebot3_manipulation_description/urdf/open_manipulator_x.urdf.xacro (robot description, xacro)
@@ -224,11 +224,17 @@
     </joint>
     <link name="${prefix}end_effector_link">
-      <visual>
-        <origin xyz="0 0 0" rpy="0 0 0"/>
-        <geometry>
-          <box size="0.01 0.01 0.01" />
-        </geometry>
-        <material name="red"/>
+       <visual>
+         <origin xyz="0 0 0" rpy="0 0 0"/>
+           <geometry>
+              <box size="0.01 0.01 0.01" />
+          </geometry>
+          <material name="red"/>
        </visual>
+       <collision>
+          <origin xyz="0 0 0" rpy="0 0 0"/>
+          <geometry>
+            <box size="0.01 0.01 0.01" />
+          </geometry>
+       </collision>
     </link>
   </xacro:macro>
